Commit message: feat(description): 对称模型资产 + 导轨/接触物理加固
- 导轨锁架构：4 导轨 position-only 命令接口（gz_ros2_control 的
  JointForceCmd 残留会永远压制位置伺服，根因见 GAZEBO_CONTROL_FIX）；
  prismatic effort 800→5000 / damping 8.0 / friction 1.0，触地冲击
  瞬态兜在 5 mm 锁定预算内
- 足底接触 kd 20→300（13 Hz 接触共振 ζ 0.04→0.55，避免振铃混叠进
  20 Hz 力控环）；足底半径 0.012→0.020，foot_tip z 同步补偿
- 对称模型：primitive 惯量选项、网格根参数化、新增对称网格 STL
  （含 collision）、Blender 生成脚本、Pinocchio/URDF 校验脚本与测试

Co-authored-by: Cursor <cursoragent@cursor.com>

File: src/dog2_description/urdf/dog2.urdf.xacro (robot description, xacro)
@@ -10,7 +10,11 @@
 <robot xmlns:xacro="http://www.ros.org/wiki/xacro" name="dog2">
   <xacro:arg name="controllers_yaml" default="$(find dog2_description)/config/ros2_controllers.yaml"/>
+  <xacro:arg name="robot_param_node" default="robot_state_publisher"/>
   <xacro:property name="controllers_yaml" value="$(arg controllers_yaml)"/>
+  <xacro:property name="robot_param_node" value="$(arg robot_param_node)"/>
   <!-- Shared constants and tiny helper macros. Keep this include before base_link and leg macros. -->
   <xacro:include filename="$(find dog2_description)/urdf/dog2_properties.xacro"/>
+  <xacro:property name="dog2_mesh_root" value="package://dog2_description/meshes"/>
+  <xacro:property name="dog2_collision_mesh_root" value="package://dog2_description/meshes/collision"/>
   <!-- Current trunk ownership: base_link is the URDF / ROS / control / Pinocchio root frame. -->
   <link name="base_link">
@@ -44,5 +48,5 @@
       <origin xyz="${0.0 - base_link_semantic_origin_x - 0.9780} ${0.0 - base_link_semantic_origin_y + 0.87203} -0.2649" rpy="0 0 0"/>
       <geometry>
-        <mesh filename="package://dog2_description/meshes/base_link.STL"/>
+        <mesh filename="${dog2_mesh_root}/base_link.STL"/>
       </geometry>
       <material name="mat_base_gray">
@@ -104,4 +108,4 @@
              foot_tip_xyz="${leg4_foot_tip_xyz}"/>
   <xacro:include filename="$(find dog2_description)/urdf/dog2_ros2_control.xacro"/>
-  <xacro:dog2_ros2_control controllers_yaml="${controllers_yaml}"/>
+  <xacro:dog2_ros2_control controllers_yaml="${controllers_yaml}" robot_param_node="${robot_param_node}"/>
 </robot>

File: src/dog2_description/urdf/dog2_leg_macro.xacro (robot description, xacro)
@@ -30,14 +30,21 @@
   <xacro:macro name="leg" params="prefix side leg_num parent_link rail_axis p_low p_up thigh_xyz shin_xyz slider_inertia_xyz foot_tip_xyz
                                  hip_xyz:='-0.016 0.0199 0.055'
-                                 knee_xyz:='-0.0233 -0.055 0.0274'">
+                                 knee_xyz:='-0.0233 -0.055 0.0274'
+                                 use_primitive_links:='false'
+                                 femur_primitive_xyz:='0 0 0' femur_primitive_rpy:='0 0 0'
+                                 femur_primitive_length:='0' femur_primitive_radius:='0'
+                                 femur_primitive_ixx:='0' femur_primitive_iyy:='0' femur_primitive_izz:='0'
+                                 tibia_primitive_xyz:='0 0 0' tibia_primitive_rpy:='0 0 0'
+                                 tibia_primitive_length:='0' tibia_primitive_radius:='0'
+                                 tibia_primitive_ixx:='0' tibia_primitive_iyy:='0' tibia_primitive_izz:='0'">
   <link name="${prefix}_rail_link">
     <inertial>
       <origin rpy="0 0 0" xyz="${slider_inertia_xyz}"/>
       <mass value="0.3"/>
-      <inertia ixx="0.0001071" ixy="0" ixz="0" iyy="8.386e-05" iyz="0" izz="7.869e-05"/>
+      <inertia ixx="${rail_ixx}" ixy="0" ixz="0" iyy="${rail_iyy}" iyz="0" izz="${rail_izz}"/>
     </inertial>
     <visual>
       <geometry>
-        <mesh filename="package://dog2_description/meshes/l${leg_num}.STL"/>
+        <mesh filename="${dog2_mesh_root}/l${leg_num}.STL"/>
       </geometry>
       <material name="mat_white"><color rgba="1 1 1 1"/></material>
@@ -45,5 +52,5 @@
     <collision>
       <geometry>
-        <mesh filename="package://dog2_description/meshes/collision/l${leg_num}_collision.STL"/>
+        <mesh filename="${dog2_collision_mesh_root}/l${leg_num}_collision.STL"/>
       </geometry>
     </collision>
@@ -83,9 +90,9 @@
       <origin rpy="0 0 0" xyz="-0.0233 -0.0383 0.000879"/>
       <mass value="0.25"/>
-      <inertia ixx="0.0001" ixy="0" ixz="0" iyy="0.0001" iyz="0" izz="0.0001"/>
+      <inertia ixx="${coxa_ixx}" ixy="0" ixz="0" iyy="${coxa_iyy}" iyz="0" izz="${coxa_izz}"/>
     </inertial>
     <visual>
       <geometry>
-        <mesh filename="package://dog2_description/meshes/l${leg_num}1.STL"/>
+        <mesh filename="${dog2_mesh_root}/l${leg_num}1.STL"/>
       </geometry>
       <material name="mat_blue"><color rgba="0.266 0.529 1 1"/></material>
@@ -93,5 +100,5 @@
     <collision>
       <geometry>
-        <mesh filename="package://dog2_description/meshes/collision/l${leg_num}1_collision.STL"/>
+        <mesh filename="${dog2_collision_mesh_root}/l${leg_num}1_collision.STL"/>
       </geometry>
     </collision>
@@ -111,29 +118,51 @@
   </joint>
   <link name="${prefix}_femur_link">
-    <inertial>
-      <origin rpy="0 0 0" xyz="${thigh_xyz}"/>
-      <mass value="0.4"/>
-      <inertia ixx="0.000666" ixy="0" ixz="0" iyy="0.000356" iyz="0.000266" izz="0.000534"/>
-    </inertial>
-    <!-- Femur mesh/collision-only rpy (not joint semantics). rf: CAD mesh flip via leg_thigh_mesh_flip_rpy. -->
-    <xacro:property name="thigh_vis_rpy" value="0 0 0"/>
-    <xacro:property name="thigh_col_rpy_eff" value="0 0 0"/>
-    <xacro:if value="${prefix == 'rf'}">
-      <xacro:property name="thigh_vis_rpy" value="${leg_thigh_mesh_flip_rpy}"/>
-      <xacro:property name="thigh_col_rpy_eff" value="${leg_thigh_mesh_flip_rpy}"/>
+    <xacro:if value="${use_primitive_links}">
+      <inertial>
+        <origin rpy="${femur_primitive_rpy}" xyz="${femur_primitive_xyz}"/>
+        <mass value="0.4"/>
+        <inertia ixx="${femur_primitive_ixx}" ixy="0" ixz="0" iyy="${femur_primitive_iyy}" iyz="0" izz="${femur_primitive_izz}"/>
+      </inertial>
+      <visual>
+        <origin rpy="${femur_primitive_rpy}" xyz="${femur_primitive_xyz}"/>
+        <geometry>
+          <cylinder radius="${femur_primitive_radius}" length="${femur_primitive_length}"/>
+        </geometry>
+        <material name="mat_femur_primitive"><color rgba="0.75 0.75 0.75 1"/></material>
+      </visual>
+      <collision>
+        <origin rpy="${femur_primitive_rpy}" xyz="${femur_primitive_xyz}"/>
+        <geometry>
+          <cylinder radius="${femur_primitive_radius}" length="${femur_primitive_length}"/>
+        </geometry>
+      </collision>
     </xacro:if>
-    <visual>
-      <origin rpy="${thigh_vis_rpy}" xyz="0 0 0"/>
-      <geometry>
-        <mesh filename="package://dog2_description/meshes/l${leg_num}11.STL"/>
-      </geometry>
-      <material name="mat_white"><color rgba="1 1 1 1"/></material>
-    </visual>
-    <collision>
-      <origin rpy="${thigh_col_rpy_eff}" xyz="0 0 0"/>
-      <geometry>
-        <mesh filename="package://dog2_description/meshes/collision/l${leg_num}11_collision.STL"/>
-      </geometry>
-    </collision>
+    <xacro:unless value="${use_primitive_links}">
+      <inertial>
+        <origin rpy="0 0 0" xyz="${thigh_xyz}"/>
+        <mass value="0.4"/>
+        <inertia ixx="${femur_ixx}" ixy="${femur_ixy}" ixz="${femur_ixz}" iyy="${femur_iyy}" iyz="${femur_iyz}" izz="${femur_izz}"/>
+      </inertial>
+      <!-- Femur mesh/collision-only rpy (not joint semantics). rf: CAD mesh flip via leg_thigh_mesh_flip_rpy. -->
+      <xacro:property name="thigh_vis_rpy" value="0 0 0"/>
+      <xacro:property name="thigh_col_rpy_eff" value="0 0 0"/>
+      <xacro:if value="${prefix == 'rf'}">
+        <xacro:property name="thigh_vis_rpy" value="${leg_thigh_mesh_flip_rpy}"/>
+        <xacro:property name="thigh_col_rpy_eff" value="${leg_thigh_mesh_flip_rpy}"/>
+      </xacro:if>
+      <visual>
+        <origin rpy="${thigh_vis_rpy}" xyz="0 0 0"/>
+        <geometry>
+          <mesh filename="${dog2_mesh_root}/l${leg_num}11.STL"/>
+        </geometry>
+        <material name="mat_white"><color rgba="1 1 1 1"/></material>
+      </visual>
+      <collision>
+        <origin rpy="${thigh_col_rpy_eff}" xyz="0 0 0"/>
+        <geometry>
+          <mesh filename="${dog2_collision_mesh_root}/l${leg_num}11_collision.STL"/>
+        </geometry>
+      </collision>
+    </xacro:unless>
   </link>
   <xacro:property name="femur_parent_link" value="${prefix}_coxa_link"/>
@@ -171,21 +200,43 @@
   </joint>
   <link name="${prefix}_tibia_link">
-    <inertial>
-      <origin rpy="0 0 0" xyz="${shin_xyz}"/>
-      <mass value="0.5"/>
-      <inertia ixx="0.004517" ixy="0.0000087" ixz="0.0000042" iyy="0.000975" iyz="-0.001769" izz="0.003666"/>
-    </inertial>
-    <visual>
-      <geometry>
-        <mesh filename="package://dog2_description/meshes/l${leg_num}111.STL"/>
-      </geometry>
-      <material name="mat_white"><color rgba="1 1 1 1"/></material>
-    </visual>
-    <!-- Collision is mesh STL (not a box/cylinder primitive). -->
-    <collision>
-      <geometry>
-        <mesh filename="package://dog2_description/meshes/collision/l${leg_num}111_collision.STL"/>
-      </geometry>
-    </collision>
+    <xacro:if value="${use_primitive_links}">
+      <inertial>
+        <origin rpy="${tibia_primitive_rpy}" xyz="${tibia_primitive_xyz}"/>
+        <mass value="0.5"/>
+        <inertia ixx="${tibia_primitive_ixx}" ixy="0" ixz="0" iyy="${tibia_primitive_iyy}" iyz="0" izz="${tibia_primitive_izz}"/>
+      </inertial>
+      <visual>
+        <origin rpy="${tibia_primitive_rpy}" xyz="${tibia_primitive_xyz}"/>
+        <geometry>
+          <cylinder radius="${tibia_primitive_radius}" length="${tibia_primitive_length}"/>
+        </geometry>
+        <material name="mat_tibia_primitive"><color rgba="0.7 0.7 0.7 1"/></material>
+      </visual>
+      <collision>
+        <origin rpy="${tibia_primitive_rpy}" xyz="${tibia_primitive_xyz}"/>
+        <geometry>
+          <cylinder radius="${tibia_primitive_radius}" length="${tibia_primitive_length}"/>
+        </geometry>
+      </collision>
+    </xacro:if>
+    <xacro:unless value="${use_primitive_links}">
+      <inertial>
+        <origin rpy="0 0 0" xyz="${shin_xyz}"/>
+        <mass value="0.5"/>
+        <inertia ixx="${tibia_ixx}" ixy="${tibia_ixy}" ixz="${tibia_ixz}" iyy="${tibia_iyy}" iyz="${tibia_iyz}" izz="${tibia_izz}"/>
+      </inertial>
+      <visual>
+        <geometry>
+          <mesh filename="${dog2_mesh_root}/l${leg_num}111.STL"/>
+        </geometry>
+        <material name="mat_white"><color rgba="1 1 1 1"/></material>
+      </visual>
+      <!-- Collision is mesh STL (not a box/cylinder primitive). -->
+      <collision>
+        <geometry>
+          <mesh filename="${dog2_collision_mesh_root}/l${leg_num}111_collision.STL"/>
+        </geometry>
+      </collision>
+    </xacro:unless>
   </link>
   <xacro:property name="tibia_parent_link" value="${prefix}_femur_link"/>
@@ -231,5 +282,5 @@
       <origin rpy="0 0 0" xyz="0 0 0"/>
       <mass value="0.05"/>
-      <inertia ixx="2.88e-06" ixy="0" ixz="0" iyy="2.88e-06" iyz="0" izz="2.88e-06"/>
+      <inertia ixx="${foot_ixx}" ixy="0" ixz="0" iyy="${foot_iyy}" iyz="0" izz="${foot_izz}"/>
     </inertial>
     <visual>

File: src/dog2_description/urdf/dog2_properties.xacro (robot description, xacro)
@@ -17,9 +17,19 @@
   <xacro:property name="tibia_effort" value="50"/>
   <xacro:property name="tibia_velocity" value="20"/>
-  <xacro:property name="prismatic_effort" value="100"/>
+  <!-- Rail lock architecture: the rails are normally clamped by a position
+       servo (rail_position_controller). The effort limit bounds the servo's
+       holding force in gz physics, so it must exceed worst-case locomotion
+       impacts or the "lock" gets shoved to the mechanical stop. -->
+  <!-- Rail lock: touchdown impulse spikes exceed 800 N through the leg chain;
+       5000 N keeps the position-servo rail transient within the 5 mm lock
+       budget and models a rigid mechanical brake. -->
+  <xacro:property name="prismatic_effort" value="5000"/>
   <xacro:property name="prismatic_velocity" value="5"/>
   <!-- Shared angle constants -->
   <xacro:property name="PI_CONST" value="3.141592653589793"/>
   <xacro:property name="half_pi" value="1.5707963267948966"/>
+  <!-- Mesh roots. Symmetric variants override these properties. -->
+  <xacro:property name="dog2_mesh_root" value="package://dog2_description/meshes"/>
+  <xacro:property name="dog2_collision_mesh_root" value="package://dog2_description/meshes/collision"/>
   <!-- 左右腿镜像：rail / coxa 固定段 / femur-tibia 轴规整层由常量表达。 -->
   <xacro:property name="leg_rail_rpy_L" value="${half_pi} 0 0"/>
@@ -34,7 +44,10 @@
   <xacro:property name="leg_thigh_mesh_flip_rpy" value="0 ${PI_CONST} 0"/>
   <!-- Right-side coxa decomposition is data-driven; preserve q=0 SE(3) if relocating mounts. -->
-  <!-- Joint passive dynamics (simulation stabilization) -->
-  <xacro:property name="prismatic_damping" value="0.25"/>
-  <xacro:property name="prismatic_friction" value="0.05"/>
+  <!-- Joint passive dynamics (simulation stabilization).
+       Rail damping/friction model a preloaded rail with brake: they absorb
+       foot-touchdown impulses so the position lock's transient excursion
+       stays within the smoke-test rail drift budget (5 mm). -->
+  <xacro:property name="prismatic_damping" value="8.0"/>
+  <xacro:property name="prismatic_friction" value="1.0"/>
   <xacro:property name="hip_damping" value="0.12"/>
   <xacro:property name="hip_friction" value="0.02"/>
@@ -111,3 +124,25 @@
   <xacro:property name="l3_inertia_xyz" value="-0.0159999123716776 0.000737036465389251 0.0261570925915838"/>
   <xacro:property name="l4_inertia_xyz" value="0.0159999123716776 0.000737036465389251 0.0261570925915838"/>
+  <!-- Leg link inertia tensors (default values, used by dog2_leg_macro.xacro) -->
+  <xacro:property name="rail_ixx" value="0.0001071"/>
+  <xacro:property name="rail_iyy" value="8.386e-05"/>
+  <xacro:property name="rail_izz" value="7.869e-05"/>
+  <xacro:property name="coxa_ixx" value="0.0001"/>
+  <xacro:property name="coxa_iyy" value="0.0001"/>
+  <xacro:property name="coxa_izz" value="0.0001"/>
+  <xacro:property name="femur_ixx" value="0.000666"/>
+  <xacro:property name="femur_ixy" value="0"/>
+  <xacro:property name="femur_ixz" value="0"/>
+  <xacro:property name="femur_iyy" value="0.000356"/>
+  <xacro:property name="femur_iyz" value="0.000266"/>
+  <xacro:property name="femur_izz" value="0.000534"/>
+  <xacro:property name="tibia_ixx" value="0.004517"/>
+  <xacro:property name="tibia_ixy" value="0.0000087"/>
+  <xacro:property name="tibia_ixz" value="0.0000042"/>
+  <xacro:property name="tibia_iyy" value="0.000975"/>
+  <xacro:property name="tibia_iyz" value="-0.001769"/>
+  <xacro:property name="tibia_izz" value="0.003666"/>
+  <xacro:property name="foot_ixx" value="2.88e-06"/>
+  <xacro:property name="foot_iyy" value="2.88e-06"/>
+  <xacro:property name="foot_izz" value="2.88e-06"/>
 </robot>

File: src/dog2_description/urdf/dog2_ros2_control.xacro (robot description, xacro)
@@ -11,5 +11,21 @@
     </joint>
   </xacro:macro>
-  <xacro:macro name="dog2_ros2_control" params="controllers_yaml">
+  <!-- Rail joints must be position-only. In gz_ros2_control 0.7.x, merely
+       exposing an effort command interface sets the joint's EFFORT control
+       bit at init, which creates a persistent JointForceCmd component in
+       gz-sim. The Fortress Physics system then ignores JointVelocityCmd (the
+       position servo) whenever JointForceCmd exists on the joint, so the
+       rail "lock" never engages and the rails stay force-free and drift.
+       Position-only also means gz's hold_joints fallback velocity-holds the
+       rails at 0 from the first physics step until the controller claims
+       them. -->
+  <xacro:macro name="dog2_rail_control_joint" params="name">
+    <joint name="${name}">
+      <command_interface name="position"/>
+      <state_interface name="position"/>
+      <state_interface name="velocity"/>
+    </joint>
+  </xacro:macro>
+  <xacro:macro name="dog2_ros2_control" params="controllers_yaml robot_param_node:=robot_state_publisher">
     <!-- ROS 2 Control -->
     <ros2_control name="GazeboSimSystem" type="system">
@@ -17,17 +33,17 @@
         <plugin>gz_ros2_control/GazeboSimSystem</plugin>
       </hardware>
-      <xacro:dog2_control_joint name="lf_rail_joint"/>
+      <xacro:dog2_rail_control_joint name="lf_rail_joint"/>
       <xacro:dog2_control_joint name="lf_coxa_joint"/>
       <xacro:dog2_control_joint name="lf_femur_joint"/>
       <xacro:dog2_control_joint name="lf_tibia_joint"/>
-      <xacro:dog2_control_joint name="lh_rail_joint"/>
+      <xacro:dog2_rail_control_joint name="lh_rail_joint"/>
       <xacro:dog2_control_joint name="lh_coxa_joint"/>
       <xacro:dog2_control_joint name="lh_femur_joint"/>
       <xacro:dog2_control_joint name="lh_tibia_joint"/>
-      <xacro:dog2_control_joint name="rh_rail_joint"/>
+      <xacro:dog2_rail_control_joint name="rh_rail_joint"/>
       <xacro:dog2_control_joint name="rh_coxa_joint"/>
       <xacro:dog2_control_joint name="rh_femur_joint"/>
       <xacro:dog2_control_joint name="rh_tibia_joint"/>
-      <xacro:dog2_control_joint name="rf_rail_joint"/>
+      <xacro:dog2_rail_control_joint name="rf_rail_joint"/>
       <xacro:dog2_control_joint name="rf_coxa_joint"/>
       <xacro:dog2_control_joint name="rf_femur_joint"/>
@@ -38,5 +54,5 @@
         <parameters>${controllers_yaml}</parameters>
         <robot_param>robot_description</robot_param>
-        <robot_param_node>robot_state_publisher</robot_param_node>
+        <robot_param_node>${robot_param_node}</robot_param_node>
       </plugin>
     </gazebo>
