Commit message: feat(locomotion): 强化 LAV 并新增独立平地 crawl 试验栈
以真实接触、双时钟和可校准质量门替换旧 smoke 假通过，并保留 crossing 栈建立可复现的安全停步基线。

Co-authored-by: Cursor <cursoragent@cursor.com>

File: src/dog2_description/urdf/dog2.urdf.xacro (robot description, xacro)
@@ -11,4 +11,7 @@
   <xacro:arg name="controllers_yaml" default="$(find dog2_description)/config/ros2_controllers.yaml"/>
   <xacro:arg name="robot_param_node" default="robot_state_publisher"/>
+  <!-- Instrumentation only: adds Gazebo contact sensors without changing links,
+       joints, geometry, inertia, limits, or ros2_control interfaces. -->
+  <xacro:arg name="enable_acceptance_contact_sensors" default="false"/>
   <xacro:property name="controllers_yaml" value="$(arg controllers_yaml)"/>
   <xacro:property name="robot_param_node" value="$(arg robot_param_node)"/>
@@ -55,4 +58,16 @@
     </visual>
   </link>
+  <xacro:if value="$(arg enable_acceptance_contact_sensors)">
+    <gazebo reference="base_link">
+      <sensor name="base_acceptance_contact" type="contact">
+        <always_on>true</always_on>
+        <update_rate>200</update_rate>
+        <contact>
+          <collision>base_link_collision</collision>
+          <topic>/dog2/gz_contact/base</topic>
+        </contact>
+      </sensor>
+    </gazebo>
+  </xacro:if>
   <!-- Leg topology macro. This include must stay before the four xacro:leg instantiations. -->
   <xacro:include filename="$(find dog2_description)/urdf/dog2_leg_macro.xacro"/>
@@ -93,18 +108,22 @@
   <xacro:leg prefix="lf" side="left" leg_num="1" parent_link="lf_leg_mount" rail_axis="${leg_rail_axis_L}" p_low="0.0" p_up="0.111"
              thigh_xyz="${leg12_thigh_xyz}" shin_xyz="${leg12_shin_xyz}" slider_inertia_xyz="${l1_inertia_xyz}"
-             foot_tip_xyz="${leg12_foot_tip_xyz}"/>
+             foot_tip_xyz="${leg12_foot_tip_xyz}"
+             enable_acceptance_contact_sensors="$(arg enable_acceptance_contact_sensors)"/>
   <xacro:leg prefix="lh" side="left" leg_num="2" parent_link="lh_leg_mount" rail_axis="${leg_rail_axis_L}" p_low="-0.111" p_up="0.0"
              thigh_xyz="${leg12_thigh_xyz}" shin_xyz="${leg12_shin_xyz}" slider_inertia_xyz="${l2_inertia_xyz}"
              hip_xyz="0.016 0.0199 0.055"
-             foot_tip_xyz="${leg12_foot_tip_xyz}"/>
+             foot_tip_xyz="${leg12_foot_tip_xyz}"
+             enable_acceptance_contact_sensors="$(arg enable_acceptance_contact_sensors)"/>
   <xacro:leg prefix="rh" side="right" leg_num="3" parent_link="rh_leg_mount" rail_axis="${leg_rail_axis_R}" p_low="-0.111" p_up="0.0"
              thigh_xyz="${leg3_thigh_xyz}" shin_xyz="${leg3_shin_xyz}" slider_inertia_xyz="${l3_inertia_xyz}"
              knee_xyz="${leg_knee_xyz_R}"
-             foot_tip_xyz="${leg3_foot_tip_xyz}"/>
+             foot_tip_xyz="${leg3_foot_tip_xyz}"
+             enable_acceptance_contact_sensors="$(arg enable_acceptance_contact_sensors)"/>
   <!-- Front-right retains its measured hip mount offset; the rest of the chain follows the shared contract. -->
   <xacro:leg prefix="rf" side="right" leg_num="4" parent_link="rf_leg_mount" rail_axis="${leg_rail_axis_R}" p_low="0.0" p_up="0.111"
              thigh_xyz="${leg4_thigh_xyz}" shin_xyz="${leg4_shin_xyz}" slider_inertia_xyz="${l4_inertia_xyz}"
              hip_xyz="0.0116 0.0199 0.055" knee_xyz="${leg_knee_xyz_R}"
-             foot_tip_xyz="${leg4_foot_tip_xyz}"/>
+             foot_tip_xyz="${leg4_foot_tip_xyz}"
+             enable_acceptance_contact_sensors="$(arg enable_acceptance_contact_sensors)"/>
   <xacro:include filename="$(find dog2_description)/urdf/dog2_ros2_control.xacro"/>
   <xacro:dog2_ros2_control controllers_yaml="${controllers_yaml}" robot_param_node="${robot_param_node}"/>

File: src/dog2_description/urdf/dog2_leg_macro.xacro (robot description, xacro)
@@ -37,5 +37,6 @@
                                  tibia_primitive_xyz:='0 0 0' tibia_primitive_rpy:='0 0 0'
                                  tibia_primitive_length:='0' tibia_primitive_radius:='0'
-                                 tibia_primitive_ixx:='0' tibia_primitive_iyy:='0' tibia_primitive_izz:='0'">
+                                 tibia_primitive_ixx:='0' tibia_primitive_iyy:='0' tibia_primitive_izz:='0'
+                                 enable_acceptance_contact_sensors:='false'">
   <link name="${prefix}_rail_link">
     <inertial>
@@ -319,8 +320,30 @@
     <maxVel>${foot_contact_max_vel}</maxVel>
     <material>Gazebo/Grey</material>
+  </gazebo>
+  <!--
+    tibia_link and foot_link are intentionally fixed-joint-lumped into the
+    surviving tibia_drive_frame.  Attach sensors directly to that surviving
+    frame and select the deterministic post-lump collision names.  This keeps
+    the default mechanics while making every sensor selector resolvable in the
+    generated SDF.
+  -->
+  <gazebo reference="${prefix}_tibia_drive_frame">
+    <xacro:if value="${enable_acceptance_contact_sensors}">
+      <sensor name="${prefix}_tibia_acceptance_contact" type="contact">
+        <always_on>true</always_on>
+        <update_rate>200</update_rate>
+        <contact>
+          <collision>${prefix}_tibia_drive_frame_fixed_joint_lump__${prefix}_tibia_link_collision</collision>
+          <topic>/dog2/gz_contact/${prefix}_tibia</topic>
+        </contact>
+      </sensor>
+    </xacro:if>
     <sensor name="${prefix}_foot_contact" type="contact">
       <always_on>true</always_on>
       <update_rate>200</update_rate>
-      <contact/>
+      <contact>
+        <collision>${prefix}_tibia_drive_frame_fixed_joint_lump__${prefix}_foot_link_collision_1</collision>
+        <topic>/dog2/gz_contact/${prefix}_foot</topic>
+      </contact>
     </sensor>
   </gazebo>

File: src/dog2_description/urdf/dog2_symmetric.urdf.xacro (robot description, xacro)
@@ -15,4 +15,7 @@
   <xacro:arg name="controllers_yaml" default="$(find dog2_description)/config/ros2_controllers.yaml"/>
   <xacro:arg name="robot_param_node" default="robot_state_publisher"/>
+  <!-- Instrumentation only: adds Gazebo contact sensors without changing links,
+       joints, geometry, inertia, limits, or ros2_control interfaces. -->
+  <xacro:arg name="enable_acceptance_contact_sensors" default="false"/>
   <xacro:property name="controllers_yaml" value="$(arg controllers_yaml)"/>
   <xacro:property name="robot_param_node" value="$(arg robot_param_node)"/>
@@ -47,4 +50,16 @@
     </visual>
   </link>
+  <xacro:if value="$(arg enable_acceptance_contact_sensors)">
+    <gazebo reference="base_link">
+      <sensor name="base_acceptance_contact" type="contact">
+        <always_on>true</always_on>
+        <update_rate>200</update_rate>
+        <contact>
+          <collision>base_link_collision</collision>
+          <topic>/dog2/gz_contact/base</topic>
+        </contact>
+      </sensor>
+    </gazebo>
+  </xacro:if>
   <!-- Leg topology macro. -->
   <xacro:include filename="$(find dog2_description)/urdf/dog2_leg_macro.xacro"/>
@@ -94,5 +109,6 @@
              tibia_primitive_xyz="${tibia_left_primitive_xyz}" tibia_primitive_rpy="${tibia_left_primitive_rpy}"
              tibia_primitive_length="${tibia_left_primitive_length}" tibia_primitive_radius="${tibia_left_primitive_radius}"
-             tibia_primitive_ixx="${tibia_left_primitive_ixx}" tibia_primitive_iyy="${tibia_left_primitive_iyy}" tibia_primitive_izz="${tibia_left_primitive_izz}"/>
+             tibia_primitive_ixx="${tibia_left_primitive_ixx}" tibia_primitive_iyy="${tibia_left_primitive_iyy}" tibia_primitive_izz="${tibia_left_primitive_izz}"
+             enable_acceptance_contact_sensors="$(arg enable_acceptance_contact_sensors)"/>
   <xacro:leg prefix="lh" side="left" leg_num="2" parent_link="lh_leg_mount" rail_axis="${leg_rail_axis_L}" p_low="-0.111" p_up="0.0"
              thigh_xyz="${leg12_thigh_xyz}" shin_xyz="${leg12_shin_xyz}" slider_inertia_xyz="${l2_inertia_xyz}"
@@ -105,5 +121,6 @@
              tibia_primitive_xyz="${tibia_left_primitive_xyz}" tibia_primitive_rpy="${tibia_left_primitive_rpy}"
              tibia_primitive_length="${tibia_left_primitive_length}" tibia_primitive_radius="${tibia_left_primitive_radius}"
-             tibia_primitive_ixx="${tibia_left_primitive_ixx}" tibia_primitive_iyy="${tibia_left_primitive_iyy}" tibia_primitive_izz="${tibia_left_primitive_izz}"/>
+             tibia_primitive_ixx="${tibia_left_primitive_ixx}" tibia_primitive_iyy="${tibia_left_primitive_iyy}" tibia_primitive_izz="${tibia_left_primitive_izz}"
+             enable_acceptance_contact_sensors="$(arg enable_acceptance_contact_sensors)"/>
   <xacro:leg prefix="rh" side="right" leg_num="3" parent_link="rh_leg_mount" rail_axis="${leg_rail_axis_R}" p_low="-0.111" p_up="0.0"
              thigh_xyz="${leg3_thigh_xyz}" shin_xyz="${leg3_shin_xyz}" slider_inertia_xyz="${l3_inertia_xyz}"
@@ -116,5 +133,6 @@
              tibia_primitive_xyz="${tibia_right_primitive_xyz}" tibia_primitive_rpy="${tibia_right_primitive_rpy}"
              tibia_primitive_length="${tibia_right_primitive_length}" tibia_primitive_radius="${tibia_right_primitive_radius}"
-             tibia_primitive_ixx="${tibia_right_primitive_ixx}" tibia_primitive_iyy="${tibia_right_primitive_iyy}" tibia_primitive_izz="${tibia_right_primitive_izz}"/>
+             tibia_primitive_ixx="${tibia_right_primitive_ixx}" tibia_primitive_iyy="${tibia_right_primitive_iyy}" tibia_primitive_izz="${tibia_right_primitive_izz}"
+             enable_acceptance_contact_sensors="$(arg enable_acceptance_contact_sensors)"/>
   <!-- Front-right: symmetric hip offset (mirrors lh), symmetric knee Z, symmetric shin/foot -->
   <xacro:leg prefix="rf" side="right" leg_num="4" parent_link="rf_leg_mount" rail_axis="${leg_rail_axis_R}" p_low="0.0" p_up="0.111"
@@ -128,5 +146,6 @@
              tibia_primitive_xyz="${tibia_right_primitive_xyz}" tibia_primitive_rpy="${tibia_right_primitive_rpy}"
              tibia_primitive_length="${tibia_right_primitive_length}" tibia_primitive_radius="${tibia_right_primitive_radius}"
-             tibia_primitive_ixx="${tibia_right_primitive_ixx}" tibia_primitive_iyy="${tibia_right_primitive_iyy}" tibia_primitive_izz="${tibia_right_primitive_izz}"/>
+             tibia_primitive_ixx="${tibia_right_primitive_ixx}" tibia_primitive_iyy="${tibia_right_primitive_iyy}" tibia_primitive_izz="${tibia_right_primitive_izz}"
+             enable_acceptance_contact_sensors="$(arg enable_acceptance_contact_sensors)"/>
   <xacro:include filename="$(find dog2_description)/urdf/dog2_ros2_control.xacro"/>
   <xacro:dog2_ros2_control controllers_yaml="${controllers_yaml}" robot_param_node="${robot_param_node}"/>
